File: Crystal_hw/Crystal.sch (KiCad schematic (older format))
At the start: 57 parts, among them SW1 BUTTON_H, U1 ADG723

Commit message: * Switch to Chibios 3.0, nothing works save UART
Parts:
- DA1: symbol GENERIC_8PIN -> Generic_8pin
- DD1: symbol STM32F405RX-64 -> STM32F405Rx-64
- HOLE1, HOLE2, HOLE3, HOLE4: symbol HOLE_METALLED -> HOLE_METALLED-RESCUE-Crystal
Changed lines of the file:
@@
 EESchema Schematic File Version 2
+LIBS:Crystal-rescue
 LIBS:adc_kl
 LIBS:Connectors_kl
@@
 LIBS:power
 LIBS:Crystal-cache
-EELAYER 27 0
+EELAYER 25 0
 EELAYER END
 $Descr A3 16535 11693
@@
 $EndComp
 $Comp
-L GENERIC_8PIN DA1
+L Generic_8pin DA1
 U 2 1 51653117
 P 5900 3000
@@
 $EndComp
 $Comp
-L GENERIC_8PIN DA1
+L Generic_8pin DA1
 U 1 1 51653126
 P 5100 2300
@@
 IN2
 $Comp
-L HOLE_METALLED HOLE1
+L HOLE_METALLED-RESCUE-Crystal HOLE1
 U 1 1 51DE9CCE
 P 14950 7200
@@
 $EndComp
 $Comp
-L HOLE_METALLED HOLE3
+L HOLE_METALLED-RESCUE-Crystal HOLE3
 U 1 1 51DE9CEA
 P 14950 7800
@@
 $EndComp
 $Comp
-L HOLE_METALLED HOLE4
+L HOLE_METALLED-RESCUE-Crystal HOLE4
 U 1 1 51DE9CF0
 P 14950 8100
@@
 $EndComp
 $Comp
-L HOLE_METALLED HOLE2
+L HOLE_METALLED-RESCUE-Crystal HOLE2
 U 1 1 51DE9CF6
 P 14950 7500
@@
 Connection ~ 1800 9100
 $Comp
-L STM32F405RX-64 DD1
+L STM32F405Rx-64 DD1
 U 1 1 51304C9D
 P 4800 7350

Commit message: + sch v4
Parts:
- removed BN1, BN2: BNC, ~, symbol BNC
- removed C1: 0.1u, symbol C
- removed C10, C11, C14, C15, C2, C3: 10u, symbol C
- removed C5: 0.01u, CAP_0603, symbol C
- removed C6: 0.1u, CAP_0603, symbol C
- removed DA4, DA5: LD1117, symbol LD1117
- removed HOLE1, HOLE2, HOLE3, HOLE4: HOLE_METALLED, symbol HOLE_METALLED-RESCUE-Crystal
- removed R1: 10K, symbol R
- removed U1: ADG723, ~, symbol ADG723
- removed XL1: CONN_3, ~, symbol CONN_3
- removed XL2: USB_MINI_B, ~, symbol USB_MINI_B
- removed XL3: ST_SWD, ~, symbol ST_SWD
- added C1, C22: 10n, Capacitors:CAP_0603, symbol Tittar_kl:C
- added C14: 0.1u, Capacitors:CAP_0603, symbol Tittar_kl:C
- added C15, C16, C17, C20, C21: 1u, Capacitors:CAP_0603, symbol Tittar_kl:C
- added DA4, DA5: MCP1700, SOT:SOT23-3A, symbol Power_kl:MCP1700
- added HOLE1, HOLE2, HOLE3, HOLE4: HOLE_METALLED, PCB:Hole3_5_out6mm, symbol pcb_details:HOLE_METALLED
- added R1: 1M, Resistors:RES_0603, symbol Tittar_kl:R
- added R8: 5R1, Resistors:RES_0603, symbol Tittar_kl:R
- added RP1, RP2: REFPOINT, PCB:REF_POINT_2MM, symbol pcb_details:REFPOINT
- added XL1: CONN_6, Connectors:PLS-6, symbol Connectors_kl:CONN_6
- added XL2: USB_MINI_B, Connectors:USBmicro_MOLEX_WM17142, symbol Connectors_kl:USB_MINI_B
- added XW1, XW2, XW3: BNC, Connectors:BNC_R, symbol Connectors_kl:BNC
- C10: renamed from C19; footprint (none) -> Capacitors:CAP_0603; symbol C -> Tittar_kl:C
- C11: renamed from C20; footprint (none) -> Capacitors:CAP_0603; symbol C -> Tittar_kl:C
- C12: renamed from C23; footprint CAP_0603 -> Capacitors:CAP_0603; symbol C -> Tittar_kl:C
- C13: renamed from C21; footprint (none) -> Capacitors:CAP_0603; symbol C -> Tittar_kl:C
- C18: renamed from C8; footprint (none) -> Capacitors:CAP_0603; symbol C -> Tittar_kl:C
- C19: renamed from C9; footprint (none) -> Capacitors:CAP_0603; symbol C -> Tittar_kl:C
- C2: renamed from C22; footprint (none) -> Capacitors:CAP_0603; symbol C -> Tittar_kl:C
- C3: renamed from C12; value 20pF -> 18pF; footprint (none) -> Capacitors:CAP_0603; symbol C -> Tittar_kl:C
- C4: renamed from C16; footprint (none) -> Capacitors:CAP_0603; symbol C -> Tittar_kl:C
- C5: renamed from C17; footprint (none) -> Capacitors:CAP_0603; symbol C -> Tittar_kl:C
- C6: renamed from C13; value 20pF -> 18pF; footprint (none) -> Capacitors:CAP_0603; symbol C -> Tittar_kl:C
- C7: renamed from C4; footprint (none) -> Capacitors:CAP_0603; symbol C -> Tittar_kl:C
- C8: renamed from C18; footprint (none) -> Capacitors:CAP_0603; symbol C -> Tittar_kl:C
- C9: renamed from C7; footprint (none) -> Capacitors:CAP_0603; symbol C -> Tittar_kl:C
- D1, D2, D3: footprint (none) -> LEDs:LED_0603; symbol LED -> Tittar_kl:LED
- DA1: value GENERIC_8PIN -> MAX4453; footprint (none) -> SOT:SOT23-8; symbol Generic_8pin -> OpAmp_kl:Generic_8pin
- DA2: renamed from DA3; footprint (none) -> SO_DIL_TSSOP:MSOP8; symbol ADS8320 -> adc_kl:ADS8320
- DA3: renamed from DA2; footprint (none) -> SO_DIL_TSSOP:MSOP8; symbol DAC8531 -> dac:DAC8531
- DD1: footprint (none) -> LQFP_TQFP:LQFP64; symbol STM32F405Rx-64 -> st_kl:STM32F405Rx-64
- R10: renamed from R7; value 200 -> 1k; footprint (none) -> Resistors:RES_0603; symbol R -> Tittar_kl:R
- R11: renamed from R8; value 200 -> 1k; footprint (none) -> Resistors:RES_0603; symbol R -> Tittar_kl:R
- R12: renamed from R3; footprint RES_0603 -> Resistors:RES_0603; symbol R -> Tittar_kl:R
- R2: footprint (none) -> Resistors:RES_0603; symbol R -> Tittar_kl:R
- R3: renamed from R4; footprint (none) -> Resistors:RES_0603; symbol R -> Tittar_kl:R
- R4: renamed from R5; value 200R -> 1k; footprint (none) -> Resistors:RES_0603; symbol R -> Tittar_kl:R
- R5, R6: renamed from R?; footprint (none) -> Resistors:RES_0603; symbol R -> Tittar_kl:R
- R7: renamed from R9; value 1k -> 10k; footprint (none) -> Resistors:RES_0603; symbol R -> Tittar_kl:R
- R9: renamed from R6; value 200 -> 1k; footprint (none) -> Resistors:RES_0603; symbol R -> Tittar_kl:R
- SW1: footprint (none) -> BtnsSwitches:BTN_4x4_SMD; symbol BUTTON_H -> Switches:BUTTON
- VCap1, VCap2: footprint (none) -> Capacitors:CAP_0603; symbol C -> Tittar_kl:C
- XTAL1: footprint CRYSTAL -> Quartz:03225C4; symbol CRYSTAL_H -> Tittar_kl:CRYSTAL_H
Connections:
- net labels added: ADC_CLK, ADC_CS, ADC_DOUT, DAC_CLK, DAC_CS, DAC_DIN, UART_RX, UART_TX
- net labels removed: CLK, CS, CSIN, D2, DIN, DOUT, IN1, IN2, RX1, S1, S2_D1, SCK, TX1
- wire segments 192 -> 227
- no-connect marks 33 -> 35
Other:
- note added: "Input\n"
- note added: "Output\n"
- note added: "Programming & debug"
- note removed: "Add it somehow"
- note removed: "Analog switch"
- note removed: "Connectors"
- note removed: "DEBUG UART\n"
- note removed: "IN\n"
- note removed: "OUT\n"
- note removed: "Programming"
- note removed: "USB"
- moved on the sheet: C10, C11, C12, C13, C2, C3, C4, C5, C6, C7, C8, C9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

Commit message: HW v20190412 in progress
Parts:
- added L1: 90R, Inductors:DLW21SN, symbol Tittar_kl:CHOKE_COIL
- added L2: BLM15AG102, Inductors:IND_0402, symbol Tittar_kl:L
- added R13: 2R0, Resistors:RES_0603, symbol Tittar_kl:R
- added R14: 10K, Resistors:RES_0603, symbol Tittar_kl:R
- added TP1, TP10, TP11, TP12, TP13, TP14, TP2, TP3, TP4, TP5, TP6, TP7, TP8, TP9: TESTPOINT, PCB:TESTPOINT_1MM, symbol pcb_details:TESTPOINT
- added U1: USBLC6, SOT:SOT23-6, symbol ESDProtection:USBLC6
- added XL3, XL4: CONN_1, Connectors:PLS-1Rnd, symbol Connectors_kl:CONN_1
- C12, C7: value 10u -> 1u
- C22: value 10n -> 2u2
- RP1, RP2: footprint PCB:REF_POINT_2MM -> PCB:REF_POINT_1MM
- XL2: value USB_MINI_B -> USB_MICRO; footprint Connectors:USBmicro_MOLEX_WM17142 -> Connectors:USBmicro_MOLEX_1050170001
- XW1, XW2, XW3: footprint Connectors:BNC_R -> Connectors:BNC2; symbol Connectors_kl:BNC -> Connectors_kl:BNC2
Connections:
- net labels added: +3v3, +5v
- net labels removed: +3.3V, +5V
- wire segments 227 -> 243
- no-connect marks 35 -> 34
Other:
- note added: "Debug\npin"
- moved on the sheet: C1, C10, C11, C12, C13, C16, C17, C18, C19, C2, C20, C21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
